Commit message: [TEST]: 修改Ignition显示效果

File: sp2_description/urdf/common/mecanum_wheel.xacro (robot description, xacro)
@@ -40,4 +40,7 @@
                         <sphere radius="${roller_radius}"/>
                     </geometry>
+                    <material name="">
+                        <color rgba="0.792156862745098 0.819607843137255 0.933333333333333 1" />
+                    </material>
                 </xacro:if>
             </collision>
@@ -77,4 +80,7 @@
                     </xacro:if>
                 </geometry>
+                <material name="">
+                    <color rgba="0.792156862745098 0.819607843137255 0.933333333333333 1" />
+                </material>
             </visual>
             <inertial>
@@ -113,5 +119,5 @@
         </xacro:unless>
     </xacro:macro>
-    <xacro:macro name="wheel_transmission" params="prefix mechanical_reduction">
+    <xacro:macro name="ros1_wheel_transmission" params="prefix mechanical_reduction">
         <transmission name="${prefix}_wheel_trans">
             <type>transmission_interface/SimpleTransmission</type>
@@ -125,3 +131,12 @@
         </transmission>
     </xacro:macro>
+    <xacro:macro name="ros2_wheel_transmission" params="prefix mechanical_reduction">
+        <transmission name="${prefix}_wheel_trans">
+            <plugin>transmission_interface/SimpleTransmission</plugin>
+            <joint name="${prefix}_wheel_joint" role="${prefix}_wheel_joint">
+                <mechanical_reduction>${mechanical_reduction}</mechanical_reduction>
+                <offset>0.0</offset>
+            </joint>
+        </transmission>
+    </xacro:macro>
 </robot>

File: sp2_description/urdf/engineer/engineer.ros2_control.xacro (robot description, xacro)
@@ -15,6 +15,6 @@
     <ros2_control name="${name}" type="system">
       <hardware>
-        <!--plugin>SP2Control/SP2Hardware</plugin-->
-        <plugin>ign_ros2_control/IgnitionSystem</plugin>
+        <plugin>SP2Control/SP2Hardware</plugin>
+        <!--plugin>ign_ros2_control/IgnitionSystem</plugin-->
         <param name="example_param_hw_start_duration_sec">0</param>
         <param name="example_param_hw_stop_duration_sec">3.0</param>
@@ -25,4 +25,8 @@
       <xacro:mecanum_joint prefix="right_front" bus_name="can0" type="rm_3508" ID="0x203"/>
       <xacro:mecanum_joint prefix="right_back" bus_name="can0" type="rm_3508" ID="0x204"/>
+      <!--xacro:ros2_wheel_transmission prefix="left_front" mechanical_reduction="19"/-->
+      <xacro:ros2_wheel_transmission prefix="left_back" mechanical_reduction="19"/>
+      <xacro:ros2_wheel_transmission prefix="right_front" mechanical_reduction="19"/>
+      <!--xacro:ros2_wheel_transmission prefix="right_back" mechanical_reduction="19"/-->
     </ros2_control>
   </xacro:macro>
