Commit message: [Fix_bugs]&&[Todo] [Fix_Bugs]: 修复麦轮读取错误的bug [Todo]: 使用静态TF发送麦轮辊子的信息

File: sp2_description/urdf/engineer/engineer.ros2_control.xacro (robot description, xacro)
@@ -1,10 +1,13 @@
 <?xml version="1.0"?>
 <robot xmlns:xacro="http://www.ros.org/wiki/xacro">
-  <xacro:macro name="mecanum_joint" params="prefix">
+  <xacro:macro name="mecanum_joint" params="prefix bus_name type ID">
       <joint name="${prefix}_wheel_joint">
-        <command_interface name="effort"/>
+			  <command_interface name="effort"/>
         <state_interface name="position"/>
         <state_interface name="velocity"/>
         <state_interface name="effort"/>
+        <param name="bus_name">${bus_name}</param>
+        <param name="type">${type}</param>
+			  <param name="ID">${ID}</param>
       </joint>
   </xacro:macro>
@@ -17,8 +20,8 @@
         <param name="example_param_hw_slowdown">100</param>
       </hardware>
-      <xacro:mecanum_joint prefix="left_front"/>
-      <xacro:mecanum_joint prefix="left_back"/>
-      <xacro:mecanum_joint prefix="right_front"/>
-      <xacro:mecanum_joint prefix="right_back"/>
+      <xacro:mecanum_joint prefix="left_front" bus_name="can0" type="rm_3508" ID="0x201"/>
+      <xacro:mecanum_joint prefix="left_back" bus_name="can0" type="rm_3508" ID="0x202"/>
+      <xacro:mecanum_joint prefix="right_front" bus_name="can0" type="rm_3508" ID="0x203"/>
+      <xacro:mecanum_joint prefix="right_back" bus_name="can0" type="rm_3508" ID="0x204"/>
     </ros2_control>
   </xacro:macro>

File: sp2_description/urdf/engineer/engineer_chassis/engineer_chassis.xacro (robot description, xacro)
@@ -4,5 +4,5 @@
      For more information, please see http://wiki.ros.org/sw_urdf_exporter -->
 <robot name="engineer_chassis" xmlns:xacro="http://www.ros.org/wiki/xacro">
-  <xacro:include filename="$(find sp2_description)/urdf/common/mecanum_wheel.xacro"/>
+  <xacro:include filename="$(find sp2_description)/urdf/common/mecanum_wheel_static.xacro"/>
   <xacro:property name="wheel_front" value="0.19727"/>
   <xacro:property name="wheel_back" value="-0.19727"/>

Commit message: [Feature]: sp2_controllers
[Format]:
1. chassis_controller文件夹结构
2. 更改轮组名back->rear
[Feature]:
1. 支持IMU_sensor_broadcaster
2. chassis_controller PID动态调整程序
3. 更新README.md

File: sp2_description/urdf/engineer/engineer.ros2_control.xacro (robot description, xacro)
@@ -15,18 +15,31 @@
     <ros2_control name="${name}" type="system">
       <hardware>
-        <plugin>SP2Control/SP2Hardware</plugin>
-        <!--plugin>ign_ros2_control/IgnitionSystem</plugin-->
+        <!--plugin>SP2Control/SP2Hardware</plugin-->
+        <plugin>ign_ros2_control/IgnitionSystem</plugin>
         <param name="example_param_hw_start_duration_sec">0</param>
         <param name="example_param_hw_stop_duration_sec">3.0</param>
         <param name="example_param_hw_slowdown">100</param>
       </hardware>
+      <!-- gz_ros2_control/gz_ros2_control/src/gz_system.cpp -->
+      <sensor name="imu_sensor">
+        <state_interface name="orientation.x"/>
+        <state_interface name="orientation.y"/>
+        <state_interface name="orientation.z"/>
+        <state_interface name="orientation.w"/>
+        <state_interface name="angular_velocity.x"/>
+        <state_interface name="angular_velocity.y"/>
+        <state_interface name="angular_velocity.z"/>
+        <state_interface name="linear_acceleration.x"/>
+        <state_interface name="linear_acceleration.y"/>
+        <state_interface name="linear_acceleration.z"/>
+      </sensor>
       <xacro:mecanum_joint prefix="left_front" bus_name="can0" type="rm_3508" ID="0x201"/>
-      <xacro:mecanum_joint prefix="left_back" bus_name="can0" type="rm_3508" ID="0x202"/>
+      <xacro:mecanum_joint prefix="left_rear" bus_name="can0" type="rm_3508" ID="0x202"/>
       <xacro:mecanum_joint prefix="right_front" bus_name="can0" type="rm_3508" ID="0x203"/>
-      <xacro:mecanum_joint prefix="right_back" bus_name="can0" type="rm_3508" ID="0x204"/>
-      <xacro:ros2_wheel_transmission prefix="left_front" mechanical_reduction="19"/>
-      <xacro:ros2_wheel_transmission prefix="left_back" mechanical_reduction="19"/>
-      <xacro:ros2_wheel_transmission prefix="right_front" mechanical_reduction="19"/>
-      <xacro:ros2_wheel_transmission prefix="right_back" mechanical_reduction="19"/>
+      <xacro:mecanum_joint prefix="right_rear" bus_name="can0" type="rm_3508" ID="0x204"/>
+      <xacro:ros2_wheel_transmission prefix="left_front" mechanical_reduction="19.203"/>
+      <xacro:ros2_wheel_transmission prefix="left_rear" mechanical_reduction="19.203"/>
+      <xacro:ros2_wheel_transmission prefix="right_front" mechanical_reduction="-19.203"/>
+      <xacro:ros2_wheel_transmission prefix="right_rear" mechanical_reduction="-19.203"/>
     </ros2_control>
   </xacro:macro>

File: sp2_description/urdf/engineer/engineer.urdf.xacro (robot description, xacro)
@@ -6,5 +6,26 @@
 	<xacro:engineer_chassis roller_type="simple"/>
 	<xacro:engineer_ros2_control name="engineer"/>
+<!-- ............................. IMU ........................................ -->
+	<link name="imu_frame"/>
+	<joint name="imu_joint" type="fixed">
+      <parent link="base_link"/>
+      <child link="imu_frame"/>
+      <origin xyz="0.0 0.0 0.0" rpy="0.0 0.0 0.0"/>
+	</joint>
+	<gazebo reference="imu_frame">
+      <sensor name="imu_sensor" type="imu">
+        <always_on>1</always_on>
+        <update_rate>100</update_rate>
+        <ignition_frame_id>imu_frame</ignition_frame_id>
+        <visualize>true</visualize>
+        <topic>imu</topic>
+      </sensor>
+	</gazebo>
+<!-- ............................. IMU ........................................ -->
   	<gazebo>
+    	  <!-- IMU plugin -->
+	  <plugin filename="ignition-gazebo-imu-system"
+        name="ignition::gazebo::systems::Imu">
+      </plugin>
     	  <!-- Joint state publisher -->
    	  <plugin filename="ign_ros2_control-system" name="ign_ros2_control::IgnitionROS2ControlPlugin">

File: sp2_description/urdf/engineer/engineer_chassis/engineer_chassis.xacro (robot description, xacro)
@@ -101,16 +101,12 @@
                          wheel_z_offset="${wheel_offset_z}"
                          reflect="-1" roller_type="${roller_type}"/>
-    <xacro:mecanum_wheel prefix="left_back" connected_to="base_link"
+    <xacro:mecanum_wheel prefix="left_rear" connected_to="base_link"
                          wheel_x_offset="${wheel_back}" wheel_y_offset="${wheel_left}"
                          wheel_z_offset="${wheel_offset_z}"
                          reflect="-1" roller_type="${roller_type}"/>
-    <xacro:mecanum_wheel prefix="right_back" connected_to="base_link"
+    <xacro:mecanum_wheel prefix="right_rear" connected_to="base_link"
                          wheel_x_offset="${wheel_back}" wheel_y_offset="${wheel_right}"
                          wheel_z_offset="${wheel_offset_z}"
                          reflect="1" roller_type="${roller_type}"/>
-    <!--xacro:wheel_transmission prefix="left_front" mechanical_reduction="19.2032"/-->
-    <!--xacro:wheel_transmission prefix="right_front" mechanical_reduction="-19.2032"/-->
-    <!--xacro:wheel_transmission prefix="left_back" mechanical_reduction="19.2032"/-->
-    <!--xacro:wheel_transmission prefix="right_back" mechanical_reduction="-19.2032"/-->
   </xacro:macro>
 <!--grappler link-->
